Commit message: model refactorisaztion and fixes

File: biotac_sim_demo/robots/shadow_hand.urdf.xacro (robot description, xacro)
@@ -36,14 +36,7 @@
 		prox_sensors="$(arg prox_sensors)" palm_sensor="$(arg palm_sensor)"
 		mounting_plate="$(arg mounting_plate)" />
-	<!-- <link name="world" /> -->
-	<!-- <joint name="rh_world_joint" type="fixed">
-		<parent link="world" />
-		<child link="rh_forearm" />
-		<origin xyz="0.0 0.0 0.0" rpy="0.0 0.0 0.0" />
-	</joint> -->
 	<gazebo>
-		<plugin filename="libsim_biotac.so" name="sim_biotac">
-			<alwaysOn>
-				true</alwaysOn>
+			<plugin filename="libsim_biotac.so" name="sim_biotac"> <!-- This works for some reason?! -->
+			<alwaysOn>true</alwaysOn>
 			<updateRate>100.0</updateRate>
 		</plugin>
